File: _autosave-Projeto_Integrador_2_Potencia.kicad_sch (KiCad schematic)
At the start: 18 parts, among them J10 Borne_CMD_Interface, J2 Vi 24V, J3 Vo 48V, J4 INA219_01x02_Socket_3.5mm, J5 INA219_01x06_Socket_2.55mm, J7 Display_01x04_Socket, J9 JST_01x02_Pin, Q1 IRF740

Commit message: Esquemático Finalizado + Começo Layout
-Precisa confirmar tamanho do Indutor
-Precisa Trocar mosfet de lugar(devido ao dissipador)
-Ao definir locais de componentes, fazer trilhas
Parts:
- renumbered ESP32_Socket_L to ESP32_Socket_L1, ESP32_Socket_R to ESP32_Socket_R1
Changed lines of the file:
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@@
 		(on_board yes)
 		(dnp no)
-		(property "Reference" "ESP32_Socket_L"
+		(property "Reference" "ESP32_Socket_L1"
 			(at 128.524 92.964 0)
 			(effects
@@
 			(project ""
 				(path "/7080dea1-265b-4d20-a61a-e2885e90866f"
-					(reference "ESP32_Socket_L")
+					(reference "ESP32_Socket_L1")
 					(unit 1)
 				)
@@
 		(on_board yes)
 		(dnp no)
-		(property "Reference" "ESP32_Socket_R"
+		(property "Reference" "ESP32_Socket_R1"
 			(at 159.258 92.456 0)
 			(effects
@@
 			(project "Projeto_Integrador_2_Potencia"
 				(path "/7080dea1-265b-4d20-a61a-e2885e90866f"
-					(reference "ESP32_Socket_R")
+					(reference "ESP32_Socket_R1")
 					(unit 1)
 				)
