File: Projeto_Integrador_2_Potencia-backups/Projeto_Integrador_2_Potencia-2024-10-19_154518/Projeto_Integrador_2_Potencia.kicad_sch (KiCad schematic)
At the start: 18 parts, among them J10 Borne_CMD_Interface, J2 Vi 24V, J3 Vo 48V, J4 INA219_01x02_Socket_3.5mm, J5 INA219_01x06_Socket_2.55mm, J7 Display_01x04_Socket, J9 JST_01x02_Pin, Q1 IRF740

Commit message: Esquemático Finalizado + Começo Layout
-Precisa confirmar tamanho do Indutor
-Precisa Trocar mosfet de lugar(devido ao dissipador)
-Ao definir locais de componentes, fazer trilhas
Parts:
- removed J10: Borne_CMD_Interface, TerminalBlock:TerminalBlock_Xinya_XY308-2.54-2P_1x02_P2.54mm_Horizontal, symbol Connector:Screw_Terminal_01x02
- removed J7: Display_01x04_Socket, Connector_PinSocket_2.54mm:PinSocket_1x04_P2.54mm_Vertical, symbol Connector:Conn_01x04_Socket
- removed J9: JST_01x02_Pin, Connector_JST:JST_EH_B2B-EH-A_1x02_P2.50mm_Vertical, symbol Connector:Conn_01x02_Pin
- added J6: Screw_Terminal_01x01, symbol Connector:Screw_Terminal_01x01
- added J9: Screw_Terminal_01x03, symbol Connector:Screw_Terminal_01x03
- C1: value 100uF -> C; footprint Capacitor_THT:CP_Radial_D10.0mm_P7.50mm -> (none)
- C2: value 22uF -> C; footprint Capacitor_THT:CP_Radial_D5.0mm_P2.50mm -> (none)
- C3: value 2.2uF -> C_Cer; footprint Capacitor_THT:C_Disc_D3.0mm_W2.0mm_P2.50mm -> (none)
- D1: footprint Diode_THT:D_A-405_P10.16mm_Horizontal -> (none)
- J1: renamed from ESP32_Socket_L; footprint Connector_PinSocket_2.54mm:PinSocket_1x15_P2.54mm_Vertical -> (none)
- J2, J3: footprint TerminalBlock:TerminalBlock_Xinya_XY308-2.54-2P_1x02_P2.54mm_Horizontal -> (none)
- J4: value INA219_01x02_Socket_3.5mm -> Conn_01x02_Socket_3.5mm; footprint TerminalBlock_4Ucon:TerminalBlock_4Ucon_1x02_P3.50mm_Horizontal -> (none)
- J5: value INA219_01x06_Socket_2.55mm -> Conn_01x06_Socket_2.55mm; footprint Connector_PinSocket_2.54mm:PinSocket_1x06_P2.54mm_Vertical -> (none)
- J8: renamed from ESP32_Socket_R; footprint Connector_PinSocket_2.54mm:PinSocket_1x15_P2.54mm_Vertical -> (none)
- L1: footprint Inductor_THT:L_Axial_L29.9mm_D14.0mm_P38.00mm_Horizontal_Vishay_IHA-105 -> (none)
- R1, R2, R3: footprint Resistor_THT:R_Axial_DIN0207_L6.3mm_D2.5mm_P10.16mm_Horizontal -> (none)
Connections:
- net 12V: now also J9.1 (Pin_1)
- net 5.2V_feedback: now also J9.3 (Pin_3)
- net GND: now also J9.2 (Pin_2)
- net pwm: now also J6.1 (Pin_1)
- net INA_Sda: now reaches J1.15 (Pin_15)
- net INA_Sda: now also J5.4 (Pin_4)
- net I2C_Scl renamed INA_Scl
- net I2C_Sda: no longer names the net of J1.11 (Pin_11)
- net I2C_Sda: no longer J5.4 (Pin_4)
Other:
- note added: "ESP32 DevKit Socket"
- note removed: "0.96 Display"
- note removed: "ESP32 DevKitV1 Socket"
